File: io_headers.kicad_sch (KiCad schematic)
At the start: 16 parts, among them J1 Conn_01x08, J10 Conn_02x04_Odd_Even, J11 Conn_02x05_Odd_Even, J12 Conn_02x04_Odd_Even, J13 Conn_02x05_Odd_Even, J14 Conn_02x03_Odd_Even, J2 Conn_01x06, J3 Conn_01x10, J4 Conn_01x08, J5 Conn_02x05_Odd_Even, J6 Conn_02x02_Odd_Even, J7 Conn_02x04_Odd_Even, J9 Conn_02x05_Odd_Even, Q1 SI1024X

Commit message: start routing
Parts:
- removed J14: Conn_02x03_Odd_Even, symbol Connector_Generic:Conn_02x03_Odd_Even
- removed J5: Conn_02x05_Odd_Even, Connector_PinHeader_2.54mm:PinHeader_2x05_P2.54mm_Vertical, symbol Connector_Generic:Conn_02x05_Odd_Even
- added J16: Conn_02x06_Odd_Even, Connector_PinHeader_2.54mm:PinHeader_2x06_P2.54mm_Vertical, symbol Connector_Generic:Conn_02x06_Odd_Even
Connections:
- net GND: now also J16.11 (Pin_11), J16.12 (Pin_12)
- net VDDIO: now also J16.1 (Pin_1), J16.2 (Pin_2)
- net X1P1A0: now also J16.3 (Pin_3)
- net X1P1B0: now also J16.4 (Pin_4)
- net X1P1C0: now also J16.5 (Pin_5)
- net X1P1D0: now also J16.6 (Pin_6)
- net X1P1G0: now also J16.8 (Pin_8)
- net X1P1K0: now also J16.9 (Pin_9)
- net X1P4A3: now also J16.10 (Pin_10)
- new net X1P1F0: J16.7 (Pin_7)

Commit message: Updated schem; Routed most of the IO
Parts:
- removed J6: Conn_02x02_Odd_Even, Connector_PinHeader_2.54mm:PinHeader_2x02_P2.54mm_Vertical, symbol Connector_Generic:Conn_02x02_Odd_Even
- added D3, D4, D5, D6: LED_GRN, LED_SMD:LED_0805_2012Metric, symbol Device:LED_Small
- added J5: Conn_01x03, symbol Connector_Generic:Conn_01x03
- added R1, R25: 4.7K, Resistor_SMD:R_0402_1005Metric, symbol Device:R_Small
- added R26, R27, R28, R29: 470, Resistor_SMD:R_0402_1005Metric, symbol Device:R_Small
- added R30, R31, R32, R33: 10K, Resistor_SMD:R_0402_1005Metric, symbol Device:R_Small
- added SW3, SW4, SW5, SW6: SW_Push, Button_Switch_SMD:SW_Push_1P1T_NO_6x6mm_H9.5mm, symbol Switch:SW_Push
- added SW7: ~, EasyEDA_Lib:SW-SMD_20P-L14.3-W5.4-P1.27-LS8.3, symbol EasyEDA_Lib:DS-10P
Connections:
- net +1.8V: now also J5.3 (Pin_3)
- net +3.3V: now also D3.2 (A), D4.2 (A), D5.2 (A), D6.2 (A), J5.1 (Pin_1)
- net GND: now also SW3.2, SW4.2, SW5.2, SW6.2
- net I2C_SCL: now also SW7.20; no longer Q1.1 (S1)
- net I2C_SCL_PU: no longer Q1.3 (D2), R14.2
- net I2C_SDA: now also SW7.19; no longer Q1.4 (S2)
- net I2C_SDA_PU: no longer Q1.6 (D1), R15.2
- net VDDIO: now also J9.3 (Pin_3), Q1.2 (G1), Q1.5 (G2), R1.1, R25.1, R30.1, R31.1, R32.1, R33.1; no longer J13.4 (Pin_4), J9.4 (Pin_4)
- net VDDIO_I2C: now also J5.2 (Pin_2); no longer Q1.2 (G1), Q1.5 (G2)
- net X0P1N0: now also J13.4 (Pin_4); no longer J13.6 (Pin_6)
- net X0P1P0: now also J13.6 (Pin_6); no longer J13.8 (Pin_8)
- net X0P4E2: now also J9.8 (Pin_8); no longer J9.7 (Pin_7)
- net X0P4E3: now also J9.7 (Pin_7); no longer J9.8 (Pin_8)
- net X0P4F1: now also J9.4 (Pin_4); no longer J9.3 (Pin_3)
- net X0P4F2: now also J9.6 (Pin_6); no longer J9.5 (Pin_5)
- net X0P4F3: now also J9.5 (Pin_5); no longer J9.6 (Pin_6)
- net X1P1A0: now also SW7.18
- net X1P1B0: now also SW7.17
- net X1P1C0: now also SW7.16
- net X1P1D0: now also SW7.15
- net X1P1F0: now also SW7.14
- net X1P1G0: now also SW7.13
- net X1P1K0: now also SW7.12
- net X1P4A3: now also SW7.11
- new net: D5.1 (K), R28.2
- new net: D6.1 (K), R29.2
- new net: D4.1 (K), R27.2
- new net: D3.1 (K), R26.2
- new net BTN0: R30.2, SW3.1, SW7.3
- new net BTN1: R31.2, SW4.1, SW7.4
- new net BTN2: R32.2, SW5.1, SW7.5
- new net BTN3: R33.2, SW6.1, SW7.6
- new net CORE_ADJ: J13.8 (Pin_8)
- new net LED0: R26.1, R27.1, R28.1, R29.1, SW7.7
- new net LED1: SW7.8
- new net LED2: SW7.9
- new net LED3: SW7.10
- new net SCL_ARD: Q1.3 (D2), R14.2
- new net SCL_XMOS: Q1.4 (S2), R1.2, SW7.1
- new net SDA_ARD: Q1.6 (D1), R15.2
- new net SDA_XMOS: Q1.1 (S1), R25.2, SW7.2
- no-connect marks 2 -> 1
Other:
- note removed: "Connect VDDIO_I2C to different voltage Disable shifter by not connect any jumper"
- moved on the sheet: J1, J10, J11, J12, J13, J16, J2, J3, J4, J7, J9, Q1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

Commit message: Finish routing
Parts:
- removed J11: Conn_02x05_Odd_Even, Connector_PinHeader_2.54mm:PinHeader_2x05_P2.54mm_Vertical, symbol Connector_Generic:Conn_02x05_Odd_Even
- added J11, J17: Conn_01x03, Connector_PinHeader_2.54mm:PinHeader_1x03_P2.54mm_Vertical, symbol Connector_Generic:Conn_01x03
- added J6: Conn_01x04, Connector_PinHeader_2.54mm:PinHeader_1x04_P2.54mm_Vertical, symbol Connector_Generic:Conn_01x04
- J5: footprint (none) -> Connector_PinHeader_2.54mm:PinHeader_1x03_P2.54mm_Vertical
Connections:
- net I2C_SCL_PU is gone; now on net SCL_ARD: J3.1 (Pin_1)
- net I2C_SDA_PU is gone; now on net SDA_ARD: J3.2 (Pin_2)
- net +1.8V: now also J11.1 (Pin_1), J11.2 (Pin_2)
- net +3.3V: now also J17.1 (Pin_1), J17.2 (Pin_2)
- net +5V: now also J6.1 (Pin_1), J6.2 (Pin_2)
- net GND: now also J7.5 (Pin_5), J7.6 (Pin_6), J11.3 (Pin_3), J17.3 (Pin_3), J6.3 (Pin_3), J6.4 (Pin_4)
- net LED0: no longer R27.1, R28.1, R29.1
- net LED1: now also R27.1
- net LED2: now also R28.1
- net LED3: now also R29.1
- net VDDIO: no longer J7.4 (Pin_4)
- net X0P1C0: no longer J7.5 (Pin_5)
- net X0P1D0: now also J7.4 (Pin_4); no longer J7.6 (Pin_6)
