File: xu316_core.kicad_sch (KiCad schematic)
At the start: 45 parts, among them U1 XU316-1024-QF60A-C32, U2 W25Q64JWUUIQ, U3 TPS62A0569PDRLR, U4 TPS62402DRCR, Y2 24MHz

Commit message: start routing
Parts:
- L1: footprint Inductor_SMD:L_0402_1005Metric -> Inductor_SMD:L_1008_2520Metric
Connections:
- net X0D04: no longer U2.2 (DO(IO1))
- net X0D05: now also U2.2 (DO(IO1))
- net +5V renamed +5V(IO)
- net +5V(IO): no longer C21.1, U3.3 (VIN), U3.5 (EN)
- new net +5V(CORE): C21.1, U3.3 (VIN), U3.5 (EN)
Other:
- note added: "Inductor FTC252012S1R0MBCA - 35mΩ"

Commit message: Updated schem; Routed most of the IO
Parts:
- removed C1: 100N, Capacitor_SMD:C_0402_1005Metric, symbol Device:C_Small
- removed R1: 4.7K, Resistor_SMD:R_0402_1005Metric, symbol Device:R_Small
- removed U2: W25Q64JWUUIQ, EasyEDA_Lib:USON-8_L4.0-W3.0-P0.80-BL_WINBOND_UU, symbol EasyEDA_Lib:W25Q64JWUUIQ
- added C38: 100N, Capacitor_SMD:C_0402_1005Metric, symbol Device:C_Small
- added R24: 4.7K, Resistor_SMD:R_0402_1005Metric, symbol Device:R_Small
- added U8: W25Q32JVSS, Package_SO:SOIC-8_5.23x5.23mm_P1.27mm, symbol Memory_Flash:W25Q32JVSS
- C2, C3: value 100N -> 22pF
- C4: value 100N -> 1uF
- R10, R9: footprint Resistor_SMD:R_0402_1005Metric -> Resistor_SMD:R_0805_2012Metric
Connections:
- net GND: now also C38.2, U8.4 (GND)
- net VDDIO: now also C38.1, R24.1, U8.8 (VCC)
- net X0D01: now also R24.2, U8.1 (~{CS})
- net X0D04: now also U8.5 (DI(IO0))
- net X0D05: now also U8.2 (DO(IO1))
- net X0D06: now also U8.3 (IO2)
- net X0D07: now also U8.7 (IO3)
- net X0D10: now also U8.6 (CLK)

Commit message: Ready to production
Parts:
- C24: footprint Capacitor_SMD:C_0402_1005Metric -> Capacitor_SMD:C_0603_1608Metric

Commit message: Updated for manufacture
Parts:
- C21: footprint Capacitor_SMD:C_0402_1005Metric -> Capacitor_SMD:C_0603_1608Metric
