File: xu316_core_board.kicad_sch (KiCad schematic)
At the start: 36 parts, among them CN1 HX JN1.27-2x10P ZZ H4.9, J15 Jack-DC, J8 Conn_01x02, SW1 RESET, U5 LMR51450, U7 NUP4114

Commit message: start routing
Parts:
- added R22, R23: 0.1, Resistor_SMD:R_0402_1005Metric, symbol Device:R_Small
- D1, D2: footprint (none) -> Diode_SMD:D_SMA
- F1: footprint (none) -> Fuse:Fuse_2512_6332Metric
- FB1: footprint (none) -> Inductor_SMD:L_0603_1608Metric
- J15: footprint (none) -> Connector_BarrelJack:BarrelJack_CUI_PJ-063AH_Horizontal
Connections:
- net +5V: now also R22.2, R23.2
- new net XU316 Core/+5V(CORE): R23.1
- new net XU316 Core/+5V(IO): R22.1
Other:
- sheet IO Headers ports: added X1P1F0; removed none
- sheet XU316 Core ports: added +5V(CORE), +5V(IO); removed +5V
- moved on the sheet: C27, C28, C29, C30, C31, C32, C33, C34, C35, C36, C37, CN1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

Commit message: Updated schem; Routed most of the IO
Parts:
- removed J8: Conn_01x02, Connector_PinHeader_2.54mm:PinHeader_1x02_P2.54mm_Vertical, symbol Connector_Generic:Conn_01x02
- removed L4: 4.7uH, Inductor_SMD:L_0402_1005Metric, symbol Device:L_Small
- added L5: 4.7uH, EasyEDA_Lib:IND-SMD_L7.0-W6.6, symbol EasyEDA_Lib:FXL0630-4R7-M
Connections:
- net DCDC_5V: now also L5.2
- net GND: now also CN1.13, CN1.15, CN1.17, CN1.19, CN1.3, CN1.5, CN1.7, CN1.9
- net at C32.2, U5.1 (SW), U5.2 (SW)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: now also L5.1
- no-connect marks 6 -> 5
Other:
- sheet IO Headers ports: added CORE_ADJ; removed none

Commit message: Finish routing
Parts:
- removed R23: 0.1, Resistor_SMD:R_0402_1005Metric, symbol Device:R_Small
- added J14, J8: Conn_01x02, Connector_PinHeader_2.54mm:PinHeader_1x02_P2.54mm_Vertical, symbol Connector_Generic:Conn_01x02
- added R34: 0.1, Resistor_SMD:R_1206_3216Metric, symbol Device:R_Small
- R22: footprint Resistor_SMD:R_0402_1005Metric -> Resistor_SMD:R_1206_3216Metric
Connections:
- net XU316 Core/+5V(IO) is gone; now on net +5V: R22.1
- net +5V: now also J14.1 (Pin_1), J8.1 (Pin_1), R34.1; no longer R22.2
- new net 5V_CORE: J8.2 (Pin_2), R34.2
- new net 5V_IO: J14.2 (Pin_2), R22.2

Commit message: Finalize the design
Parts:
- R22, R34: JLCPart (none) -> C411236
Changed lines of the file:
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@@
+			)
+		)
+		(property "JLCPart" "C411236"
+			(at 50.8 153.67 0)
+			(effects
+				(font
+					(size 1.27 1.27)
+				)
+				(hide yes)
 			)
 		)
@@
 			(at 50.8 139.7 0)
 			(effects
+				(font
+					(size 1.27 1.27)
+				)
+				(hide yes)
+			)
+		)
+		(property "JLCPart" "C411236"
+			(at 50.8 139.7 0)
+			(effects

Commit message: Ready to production
Parts:
- removed C35: 33U, Capacitor_SMD:C_0402_1005Metric, symbol Device:C_Small
- C34: footprint Capacitor_SMD:C_0402_1005Metric -> Capacitor_SMD:CP_Elec_4x5.4; JLCParts (none) -> C53200078
Connections:
- net +1.8V: now also CN1.2; no longer CN1.1
- net GND: now also CN1.10, CN1.14, CN1.16, CN1.18, CN1.20, CN1.4, CN1.6, CN1.8; no longer CN1.13, CN1.15, CN1.17, CN1.19, CN1.3, CN1.5, CN1.7, CN1.9
- net RST_N: now also CN1.9; no longer CN1.10
- net TCK: now also CN1.3; no longer CN1.4
- net TDI: now also CN1.7; no longer CN1.8
- net TDO: now also CN1.5; no longer CN1.6
- net TMS: now also CN1.1; no longer CN1.2
- net VDDIO: now also CN1.12; no longer CN1.11
- net XL_DN0: now also CN1.13; no longer CN1.14
- net XL_DN1: now also CN1.11; no longer CN1.12
- net XL_UP0: now also CN1.15; no longer CN1.16
- net XL_UP1: now also CN1.17; no longer CN1.18
Other:
- moved on the sheet: C34
Changed lines of the file:
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@@
 	)
 	(junction
-		(at 274.32 147.32)
-		(diameter 0)
-		(color 0 0 0 0)
-	)
-	(junction
 		(at 274.32 139.7)
 		(diameter 0)
@@
 	)
 	(junction
-		(at 270.51 139.7)
-		(diameter 0)
-		(color 0 0 0 0)
-	)
-	(junction
 		(at 181.61 133.35)
 		(diameter 0)
@@
 	(wire
 		(pts
-			(xy 270.51 139.7) (xy 261.62 139.7)
+			(xy 261.62 139.7) (xy 274.32 139.7)
 		)
 		(stroke
@@
 	(wire
 		(pts
-			(xy 274.32 147.32) (xy 270.51 147.32)
-		)
-		(stroke
-			(width 0)
-			(type default)
-		)
-	)
-	(wire
-		(pts
 			(xy 129.54 30.48) (xy 149.86 30.48)
 		)
@@
 	(wire
 		(pts
-			(xy 274.32 139.7) (xy 270.51 139.7)
-		)
-		(stroke
-			(width 0)
-			(type default)
-		)
-	)
-	(wire
-		(pts
 			(xy 251.46 151.13) (xy 251.46 152.4)
 		)
@@
 	(wire
 		(pts
-			(xy 270.51 147.32) (xy 270.51 146.05)
+			(xy 274.32 147.32) (xy 274.32 146.05)
 		)
 		(stroke
@@
 	(wire
 		(pts
-			(xy 279.4 140.97) (xy 279.4 139.7)
-		)
-		(stroke
-			(width 0)
-			(type default)
-		)
-	)
-	(wire
-		(pts
 			(xy 76.2 77.47) (xy 114.3 77.47)
 		)
@@
 	(wire
 		(pts
-			(xy 279.4 139.7) (xy 274.32 139.7)
-		)
-		(stroke
-			(width 0)
-			(type default)
-		)
-	)
-	(wire
-		(pts
 			(xy 91.44 144.78) (xy 91.44 146.05)
 		)
@@
 	(wire
 		(pts
-			(xy 270.51 139.7) (xy 270.51 140.97)
+			(xy 274.32 139.7) (xy 274.32 140.97)
 		)
 		(stroke
@@
 	(wire
 		(pts
-			(xy 279.4 146.05) (xy 279.4 147.32)
-		)
-		(stroke
-			(width 0)
-			(type default)
-		)
-	)
-	(wire
-		(pts
 			(xy 50.8 144.78) (xy 50.8 142.24)
 		)
@@
 	(wire
 		(pts
-			(xy 279.4 147.32) (xy 274.32 147.32)
-		)
-		(stroke
-			(width 0)
-			(type default)
-		)
-	)
-	(wire
-		(pts
 			(xy 261.62 152.4) (xy 254 152.4)
 		)
@@
 	(symbol
 		(lib_id "Device:C_Small")
-		(at 270.51 143.51 0)
+		(at 274.32 143.51 0)
 		(mirror y)
 		(unit 1)
@@
 		(dnp no)
 		(property "Reference" "C34"
-			(at 267.97 142.2462 0)
+			(at 271.78 142.2462 0)
 			(effects
 				(font
@@
 		)
 		(property "Value" "33U"
-			(at 267.97 144.7862 0)
+			(at 271.78 144.7862 0)
 			(effects
 				(font
@@
 			)
 		)
-		(property "Footprint" "Capacitor_SMD:C_0402_1005Metric"
-			(at 270.51 143.51 0)
+		(property "Footprint" "Capacitor_SMD:CP_Elec_4x5.4"
+			(at 274.32 143.51 0)
 			(effects
 				(font
@@
 		)
 		(property "Datasheet" "~"
-			(at 270.51 143.51 0)
+			(at 274.32 143.51 0)
 			(effects
 				(font
@@
 		)
 		(property "Description" "Unpolarized capacitor, small symbol"
-			(at 270.51 143.51 0)
+			(at 274.32 143.51 0)
+			(effects
+				(font
+					(size 1.27 1.27)
+				)
+				(hide yes)
+			)
+		)
+		(property "JLCParts" "C53200078"
+			(at 274.32 143.51 0)
 			(effects
 				(font
@@
 	)
 	(symbol
-		(lib_id "Device:C_Small")
-		(at 279.4 143.51 0)
-		(mirror y)
-		(unit 1)
-		(exclude_from_sim no)
-		(in_bom yes)
-		(on_board yes)
-		(dnp no)
-		(property "Reference" "C35"
-			(at 276.86 142.2462 0)
-			(effects
-				(font
-					(size 1.27 1.27)
-				)
-				(justify left)
-			)
-		)
-		(property "Value" "33U"
-			(at 276.86 144.7862 0)
-			(effects
-				(font
-					(size 1.27 1.27)
-				)
-				(justify left)
-			)
-		)
-		(property "Footprint" "Capacitor_SMD:C_0402_1005Metric"
-			(at 279.4 143.51 0)
-			(effects
-				(font
-					(size 1.27 1.27)
-				)
-				(hide yes)
-			)
-		)
-		(property "Datasheet" "~"
-			(at 279.4 143.51 0)
-			(effects
-				(font
-					(size 1.27 1.27)
-				)
-				(hide yes)
-			)
-		)
-		(property "Description" "Unpolarized capacitor, small symbol"
-			(at 279.4 143.51 0)
-			(effects
-				(font
-					(size 1.27 1.27)
-				)
-				(hide yes)
-			)
-		)
-		(pin "1"
-		)
-		(pin "2"
-		)
-		(instances
-			(project "xu316_core_board"
-				(path "/65cc93e9-be84-4175-93a1-dc6d5ec502ad"
-					(reference "C35")
-					(unit 1)
-				)
-			)
-		)
-	)
-	(symbol
 		(lib_id "Device:R_Small")
 		(at 247.65 76.2 270)
@@
 		(lib_id "EasyEDA_Lib:HX JN1.27-2X10P ZZ H4.9")
 		(at 107.95 146.05 0)
+		(mirror y)
 		(unit 1)
 		(exclude_from_sim no)

Commit message: Updated for manufacture
Parts:
- C30: footprint Capacitor_SMD:C_0402_1005Metric -> Capacitor_SMD:C_1206_3216Metric
- J15: footprint Connector_BarrelJack:BarrelJack_CUI_PJ-063AH_Horizontal -> Connector_BarrelJack:BarrelJack_GCT_DCJ200-10-A_Horizontal
Changed lines of the file:
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@@
 			)
 		)
-		(property "Footprint" "Capacitor_SMD:C_0402_1005Metric"
+		(property "Footprint" "Capacitor_SMD:C_1206_3216Metric"
 			(at 181.61 137.16 0)
 			(effects
@@
 			)
 		)
-		(property "Footprint" "Connector_BarrelJack:BarrelJack_CUI_PJ-063AH_Horizontal"
+		(property "Footprint" "Connector_BarrelJack:BarrelJack_GCT_DCJ200-10-A_Horizontal"
 			(at 182.88 155.956 0)
 			(effects
